Commit message: [mini_quadrotor] add links and joints related to cameras and modify depth camera plugin type

File: robots/mini_quadrotor/urdf/infratable/robot.gazebo.xacro (robot description, xacro)
@@ -12,35 +12,49 @@
     <mu2>0.1</mu2>
   </gazebo>
-  <!-- link for cameras -->
-  <joint name="realsence_link_joint" type="fixed">
+  <joint name="camera_link_joint" type="fixed">
     <parent link="main_body"/>
-    <child link="realsence_link"/>
+    <child link="camera_link"/>
     <origin xyz="0.1 0 0" rpy="0 0 0"/>
   </joint>
-  <link name="realsence_link"/>
-  <!-- for depth  -->
-  <joint name="realsence_depth_joint" type="fixed">
+  <link name="camera_link"/>
+  <joint name="camera_joint" type="fixed">
     <origin xyz="0 0 0" rpy="0 0 0"/>
-    <parent link="realsence_link"/>
-    <child link="realsence_depth_frame" />
+    <parent link="camera_link"/>
+    <child link="camera_rgb_frame"/>
   </joint>
-  <link name="realsence_depth_frame"/>
+  <link name="camera_rgb_frame"/>
+  <joint name="camera_rgb_optical_joint" type="fixed">
+    <origin xyz="0 0 0" rpy="${-pi / 2.0} 0 ${-pi / 2.0}" />
+    <parent link="camera_rgb_frame" />
+    <child link="camera_rgb_optical_frame" />
+  </joint>
+  <link name="camera_rgb_optical_frame"/>
+  <joint name="camera_depth_joint" type="fixed">
+    <origin xyz="0 0 0" rpy="0 0 0" />
+    <parent link="camera_link" />
+    <child link="camera_depth_frame" />
+  </joint>
+  <link name="camera_depth_frame"/>
+  <joint name="camera_depth_optical_joint" type="fixed">
+    <origin xyz="0 0 0" rpy="${-pi / 2.0} 0 ${-pi / 2.0}" />
+    <parent link="camera_depth_frame" />
+    <child link="camera_depth_optical_frame" />
+  </joint>
+  <link name="camera_depth_optical_frame"/>
   <!-- gazebo plugin -->
-  <gazebo reference="realsence_depth_frame">
-    <sensor type="depth" name="realsence_camera">
+  <gazebo reference="camera_link">
+    <sensor type="depth" name="camera">
       <always_on>true</always_on>
-      <visualize>false</visualize>
       <update_rate>20.0</update_rate>
-      <camera name="head">
-        <horizontal_fov>1.2</horizontal_fov>
-        <!--vertical_fov>1.14319</vertical_fov-->
+      <camera>
+        <horizontal_fov>${60.0*pi/180.0}</horizontal_fov>
         <image>
-          <width>1200</width>
-          <height>800</height>
-          <format>R8G8B8</format>
+          <format>B8G8R8</format>
+          <width>640</width>
+          <height>480</height>
         </image>
         <clip>
-          <near>0.02</near>
-          <far>300</far>
+          <near>0.05</near>
+          <far>8.0</far>
         </clip>
         <noise>
@@ -51,25 +65,20 @@
       </camera>
       <plugin name="depth_camera" filename="libgazebo_ros_depth_camera.so">
-        <baseline>0.06</baseline>
+        <cameraName>camera</cameraName>
         <alwaysOn>true</alwaysOn>
-        <updateRate>10.0</updateRate>
-        <imageTopicName>depth_camera/color/image_raw</imageTopicName>
-        <cameraInfoTopicName>depth_camera/color/camera_info</cameraInfoTopicName>
-        <pointCloudTopicName>depth_camera/depth/points</pointCloudTopicName>
-        <depthImageTopicName>depth_camera/depth/image_raw</depthImageTopicName>
-        <depthImageCameraInfoTopicName>depth_camera/depth/camera_info</depthImageCameraInfoTopicName>
-        <frameName>realsence_depth_frame</frameName>
-        <pointCloudCutoff>0.5</pointCloudCutoff>
-        <cameraName>realsence</cameraName>
-        <distortionK1>0.05</distortionK1>
-        <distortionK2>-0.05</distortionK2>
-        <distortionK3>0</distortionK3>
-        <distortionT1>0</distortionT1>
-        <distortionT2>0</distortionT2>
-        <CxPrime>0</CxPrime>
-        <Cx>0</Cx>
-        <Cy>0</Cy>
-        <focalLength>0</focalLength>
-        <hackBaseline>0.12</hackBaseline>
+        <updateRate>10</updateRate>
+        <imageTopicName>color/image_raw</imageTopicName>
+        <depthImageTopicName>depth/image_raw</depthImageTopicName>
+        <pointCloudTopicName>depth/points</pointCloudTopicName>
+        <cameraInfoTopicName>color/camera_info</cameraInfoTopicName>
+        <depthImageCameraInfoTopicName>depth/camera_info</depthImageCameraInfoTopicName>
+        <frameName>$(arg robot_name)/camera_depth_optical_frame</frameName>
+        <baseline>0.1</baseline>
+        <distortionK1>0.0</distortionK1>
+        <distortionK2>0.0</distortionK2>
+        <distortionK3>0.0</distortionK3>
+        <distortionT1>0.0</distortionT1>
+        <distortionT2>0.0</distortionT2>
+        <pointCloudCutoff>0.4</pointCloudCutoff>
       </plugin>
     </sensor>
