Commit message: add fixed-cant Hugmy flight simulation model

File: robots/hugmy/urdf/hugmy2.urdf.xacro (robot description, xacro)
@@ -5,4 +5,9 @@
   <baselink name="fc" />
   <thrust_link name="thrust" />
+  <!-- Set by the fixed-arm flight-simulation wrapper.  Normal URDF use keeps
+       the articulated joints unchanged. -->
+  <xacro:arg name="fixed_arms" default="false" />
+  <xacro:property name="fixed_arms_enabled" value="$(arg fixed_arms)" />
+  <xacro:arg name="body_mesh" default="package://hugmy/urdf/mesh/body_with_face.STL" />
   <!-- kinematics [m] -->
   <xacro:property name="rotor_x" value="0.08479" />
@@ -11,4 +16,8 @@
   <!-- <xacro:property name="rotor_z" value="0.055" /> -->
   <xacro:property name="rotor_z" value="0.0024" />
+  <!-- Fixed tangential cant selected by fixed_tilt_results_2.  With the
+       HUGMY arm frame convention, -direction about local X makes the
+       geometric yaw moment oppose the positive-thrust reaction torque. -->
+  <xacro:property name="rotor_cant" value="${6.5*pi/180.0}" />
   <!-- dynamics -->
   <m_f_rate value="-0.0068" /> <!-- drag torque rate -->
@@ -47,5 +56,5 @@
       <parent link="link_${id}_rotor"/>
       <child link="thrust${id}"/>
-      <origin rpy="0 0 0" xyz="-0.020 0.000 0.0369"/>
+      <origin rpy="${-direction*rotor_cant} 0 0" xyz="-0.020 0.000 0.0369"/>
       <!-- <origin rpy="0 0 0" xyz="${x} ${y} ${z}"/> -->
       <axis xyz="0 0 ${direction}"/>
@@ -135,5 +144,5 @@
       <origin rpy="0 0 0" xyz="0 0 0"/>
       <geometry>
-        <mesh filename="package://hugmy/urdf/mesh/body_with_face.STL" />
+        <mesh filename="$(arg body_mesh)" />
       </geometry>
     </visual>
@@ -228,8 +237,8 @@
     </link>
     <!-- joint -->
-    <joint name="joint_${id}_1" type="revolute">
+    <joint name="joint_${id}_1" type="${'fixed' if fixed_arms_enabled else 'revolute'}">
       <parent link="main_body"/>
       <child link="link_${id}_1"/>
-      <origin rpy="0 0 ${3*pi/4 - pi/2*(id-1)}" xyz="${base_offset}"/>
+      <origin rpy="0 0 ${-3*pi/4 + pi/2*(id-1)}" xyz="${base_offset}"/>
       <axis xyz="0 -1 0"/>
       <limit lower="0" upper="0.8727" effort="10" velocity="1.0"/>
@@ -237,5 +246,5 @@
       <dynamics damping="0.002" friction="0.2"/>
     </joint>
-    <joint name="joint_${id}_2" type="revolute">
+    <joint name="joint_${id}_2" type="${'fixed' if fixed_arms_enabled else 'revolute'}">
       <parent link="link_${id}_1"/>
       <child link="link_${id}_2"/>
@@ -246,5 +255,5 @@
       <dynamics damping="0.002" friction="0.2"/>
     </joint>
-    <joint name="joint_${id}_3" type="revolute">
+    <joint name="joint_${id}_3" type="${'fixed' if fixed_arms_enabled else 'revolute'}">
       <parent link="link_${id}_2"/>
       <child link="link_${id}_rotor"/>
@@ -255,5 +264,5 @@
       <dynamics damping="0.002" friction="0.2"/>
     </joint>
-    <joint name="joint_${id}_4" type="revolute">
+    <joint name="joint_${id}_4" type="${'fixed' if fixed_arms_enabled else 'revolute'}">
       <parent link="link_${id}_rotor"/>
       <child link="link_${id}_4"/>
@@ -264,5 +273,5 @@
       <dynamics damping="0.002" friction="0.2"/>
     </joint>
-    <joint name="joint_${id}_5" type="revolute">
+    <joint name="joint_${id}_5" type="${'fixed' if fixed_arms_enabled else 'revolute'}">
       <parent link="link_${id}_4"/>
       <child link="link_${id}_end"/>
@@ -273,4 +282,8 @@
       <dynamics damping="0.002" friction="0.2"/>
     </joint>
+    <!-- Fixed joints are merged by Gazebo.  Do not register effort
+         transmissions for them: gazebo_ros_control would otherwise wait for
+         joint handles which no longer exist. -->
+    <xacro:if value="${not fixed_arms_enabled}">
     <transmission name="joint_${id}_1_tran">
       <type>transmission_interface/SimpleTransmission</type>
@@ -323,4 +336,5 @@
       </actuator>
     </transmission>
+    </xacro:if>
   </xacro:macro>
   <!-- Main body links and repeated arms -->
@@ -329,8 +343,8 @@
   <!-- <xacro:arm_module id="3" base_offset="-0.05391 0.0175 -0.039"/> -->
   <!-- <xacro:arm_module id="4" base_offset="-0.0175 -0.05391 -0.039"/> -->
-  <xacro:arm_module id="1" base_offset=" 0.03812 -0.03812 -0.039"/>
-  <xacro:arm_module id="2" base_offset="-0.03812 -0.03812 -0.039"/>
-  <xacro:arm_module id="3" base_offset="-0.03812  0.03812 -0.039"/>
-  <xacro:arm_module id="4" base_offset=" 0.03812  0.03812 -0.039"/>
+  <xacro:arm_module id="1" base_offset=" 0.03812  0.03812 -0.039"/>
+  <xacro:arm_module id="2" base_offset="-0.03812  0.03812 -0.039"/>
+  <xacro:arm_module id="3" base_offset="-0.03812 -0.03812 -0.039"/>
+  <xacro:arm_module id="4" base_offset=" 0.03812 -0.03812 -0.039"/>
   <!-- spinal -->
   <xacro:extra_module name = "fc" parent = "main_body" visible = "0" >
@@ -409,8 +423,8 @@
   <!-- </joint> -->
   <!-- propellers -->
-  <xacro:propeller_module id = "1" x = "${rotor_x}" y = "${rotor_y}" z = "${rotor_z}" direction = "-1" />
-  <xacro:propeller_module id = "2" x = "${-rotor_x}" y = "${rotor_y}" z = "${rotor_z}" direction = "1" />
-  <xacro:propeller_module id = "3" x = "${-rotor_x}" y = "${-rotor_y}" z = "${rotor_z}" direction = "-1" />
-  <xacro:propeller_module id = "4" x = "${rotor_x}" y = "${-rotor_y}" z = "${rotor_z}"  direction = "1" />
+  <xacro:propeller_module id = "1" x = "${rotor_x}" y = "${rotor_y}" z = "${rotor_z}" direction = "1" />
+  <xacro:propeller_module id = "2" x = "${-rotor_x}" y = "${rotor_y}" z = "${rotor_z}" direction = "-1" />
+  <xacro:propeller_module id = "3" x = "${-rotor_x}" y = "${-rotor_y}" z = "${rotor_z}" direction = "1" />
+  <xacro:propeller_module id = "4" x = "${rotor_x}" y = "${-rotor_y}" z = "${rotor_z}"  direction = "-1" />
   <!-- propellers -->
   <!-- <xacro:propeller_module id = "1" x = "${-rotor_x}" y = "${-rotor_y}" z = "${rotor_z}" direction = "1" /> -->
